File: KiCAD/CPU/ALU.kicad_sch (KiCad schematic)
At the start: 14 parts, among them U13 74LS181, U14 74LS182, U15 74LS181, U16 74LS181, U17 74LS181, U18 74LS244, U19 74LS244, U20 74LS20, U21 74LS86, U22 74LS86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

Commit message: readme
Connections:
- net F0: now also U24.2 (P0)
- net F1: now also U24.4 (P1)
- net F10: now also U25.6 (P2)
- net F11: now also U25.8 (P3)
- net F12: now also U25.11 (P4)
- net F13: now also U25.13 (P5)
- net F14: now also U25.15 (P6)
- net F15: now also U25.17 (P7)
- net F2: now also U24.6 (P2)
- net F3: now also U24.8 (P3)
- net F4: now also U24.11 (P4)
- net F5: now also U24.13 (P5)
- net F6: now also U24.15 (P6)
- net F7: now also U24.17 (P7)
- net F8: now also U25.2 (P0)
- net F9: now also U25.4 (P1)
- net OUT0: no longer U24.2 (P0)
- net OUT1: no longer U24.4 (P1)
- net OUT10: no longer U25.6 (P2)
- net OUT11: no longer U25.8 (P3)
- net OUT12: no longer U25.11 (P4)
- net OUT13: no longer U25.13 (P5)
- net OUT14: no longer U25.15 (P6)
- net OUT15: no longer U25.17 (P7)
- net OUT2: no longer U24.6 (P2)
- net OUT3: no longer U24.8 (P3)
- net OUT4: no longer U24.11 (P4)
- net OUT5: no longer U24.13 (P5)
- net OUT6: no longer U24.15 (P6)
- net OUT7: no longer U24.17 (P7)
- net OUT8: no longer U25.2 (P0)
- net OUT9: no longer U25.4 (P1)
- net VCC: now also U24.20 (VCC), U25.20 (VCC)
- net ~{OE}: now reaches U19.1 (OEa)
- net ~{OE}: now also U18.1 (OEa), U18.19 (OEb), U19.19 (OEb)
Other:
- moved on the sheet: U24, U25
