File: KiCAD/CPU/CPU.kicad_sch (KiCad schematic)
At the start: 0 parts

Commit message: readme
Other:
- added sheet C (REG.kicad_sch)
- added sheet IR (REG.kicad_sch)
- sheet ALU ports: added ~{OE}; removed none
- note added: "(A) IN bus"
- note added: "(B) OUT bus"
