File: KiCAD/CPU/CPU.kicad_sch (KiCad schematic)
At the start: 0 parts

Commit message: small updates
Other:
- added sheet uSEQ (decode.kicad_sch)
- sheet A ports: added ~{EN}; removed CK
- sheet B ports: added ~{EN}; removed CK
- sheet C ports: added ~{EN}; removed CK
- sheet IR ports: added ~{EN}; removed CK
- sheet MAR ports: added ~{EN}; removed CK
- sheet PC ports: added none; removed CK
Changed lines of the file:
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@@
+	)
+	(junction
+		(at 125.73 71.12)
+		(diameter 0)
+		(color 0 0 0 0)
 	)
 	(junction
@@
 	)
 	(junction
-		(at 125.73 71.12)
-		(diameter 0)
-		(color 0 0 0 0)
-	)
-	(junction
 		(at 43.18 110.49)
 		(diameter 0)
@@
 	(wire
 		(pts
-			(xy 78.74 58.42) (xy 78.74 60.96)
+			(xy 76.2 58.42) (xy 76.2 60.96)
 		)
 		(stroke
@@
 		)
 	)
+	(wire
+		(pts
+			(xy 72.39 90.17) (xy 116.84 90.17)
+		)
+		(stroke
+			(width 0)
+			(type default)
+		)
+	)
+	(wire
+		(pts
+			(xy 72.39 73.66) (xy 116.84 73.66)
+		)
+		(stroke
+			(width 0)
+			(type default)
+		)
+	)
 	(bus
 		(pts
@@
 		)
 	)
-	(bus
-		(pts
-			(xy 83.82 105.41) (xy 83.82 97.79)
+	(wire
+		(pts
+			(xy 72.39 113.03) (xy 80.01 113.03)
+		)
+		(stroke
+			(width 0)
+			(type default)
+		)
+	)
+	(bus
+		(pts
+			(xy 83.82 105.41) (xy 83.82 96.52)
 		)
 		(stroke
@@
 		)
 	)
+	(wire
+		(pts
+			(xy 80.01 93.98) (xy 116.84 93.98)
+		)
+		(stroke
+			(width 0)
+			(type default)
+		)
+	)
+	(wire
+		(pts
+			(xy 80.01 113.03) (xy 80.01 93.98)
+		)
+		(stroke
+			(width 0)
+			(type default)
+		)
+	)
+	(wire
+		(pts
+			(xy 83.82 62.23) (xy 83.82 68.58)
+		)
+		(stroke
+			(width 0)
+			(type default)
+		)
+	)
 	(bus
 		(pts
@@
 	(bus
 		(pts
-			(xy 125.73 71.12) (xy 125.73 97.79)
+			(xy 125.73 71.12) (xy 125.73 96.52)
 		)
 		(stroke
@@
 	(wire
 		(pts
-			(xy 72.39 58.42) (xy 78.74 58.42)
+			(xy 115.57 107.95) (xy 124.46 107.95)
+		)
+		(stroke
+			(width 0)
+			(type default)
+		)
+	)
+	(wire
+		(pts
+			(xy 72.39 58.42) (xy 76.2 58.42)
 		)
 		(stroke
@@
 	(bus
 		(pts
-			(xy 83.82 97.79) (xy 125.73 97.79)
+			(xy 83.82 96.52) (xy 125.73 96.52)
+		)
+		(stroke
+			(width 0)
+			(type default)
+		)
+	)
+	(wire
+		(pts
+			(xy 87.63 62.23) (xy 83.82 62.23)
+		)
+		(stroke
+			(width 0)
+			(type default)
+		)
+	)
+	(wire
+		(pts
+			(xy 107.95 39.37) (xy 118.11 39.37)
+		)
+		(stroke
+			(width 0)
+			(type default)
+		)
+	)
+	(bus
+		(pts
+			(xy 154.94 35.56) (xy 167.64 35.56)
 		)
 		(stroke
@@
 		)
 	)
+	(wire
+		(pts
+			(xy 83.82 68.58) (xy 116.84 68.58)
+		)
+		(stroke
+			(width 0)
+			(type default)
+		)
+	)
 	(bus
 		(pts
@@
 			(width 0)
 			(type default)
+		)
+	)
+	(label "~{C_OE}"
+		(at 116.84 90.17 180)
+		(effects
+			(font
+				(size 1.27 1.27)
+			)
+			(justify right bottom)
+		)
+	)
+	(label "~{B_OE}"
+		(at 116.84 73.66 180)
+		(effects
+			(font
+				(size 1.27 1.27)
+			)
+			(justify right bottom)
+		)
+	)
+	(label "~{PC_OE}"
+		(at 118.11 39.37 180)
+		(effects
+			(font
+				(size 1.27 1.27)
+			)
+			(justify right bottom)
+		)
+	)
+	(label "~{A_OE}"
+		(at 116.84 93.98 180)
+		(effects
+			(font
+				(size 1.27 1.27)
+			)
+			(justify right bottom)
+		)
+	)
+	(label "~{RAM_OE}"
+		(at 116.84 68.58 180)
+		(effects
+			(font
+				(size 1.27 1.27)
+			)
+			(justify right bottom)
+		)
+	)
+	(label "~{ALU_OE}"
+		(at 124.46 107.95 180)
+		(effects
+			(font
+				(size 1.27 1.27)
+			)
+			(justify right bottom)
 		)
 	)
 	(symbol
 		(lib_id "power:GND")
-		(at 78.74 60.96 0)
+		(at 76.2 60.96 0)
 		(unit 1)
 		(body_style 1)
@@
 		(fields_autoplaced yes)
 		(property "Reference" "#PWR062"
-			(at 78.74 67.31 0)
+			(at 76.2 67.31 0)
 			(hide yes)
 			(show_name no)
@@
 		)
 		(property "Value" "GND"
-			(at 78.74 66.04 0)
+			(at 76.2 66.04 0)
 			(show_name no)
 			(do_not_autoplace no)
@@
 		)
 		(property "Footprint" ""
-			(at 78.74 60.96 0)
+			(at 76.2 60.96 0)
 			(hide yes)
 			(show_name no)
@@
 		)
 		(property "Datasheet" ""
-			(at 78.74 60.96 0)
+			(at 76.2 60.96 0)
 			(hide yes)
 			(show_name no)
@@
 		)
 		(property "Description" "Power symbol creates a global label with name \"GND\" , ground"
-			(at 78.74 60.96 0)
+			(at 76.2 60.96 0)
 			(hide yes)
 			(show_name no)
@@
 			)
 		)
-		(pin "CK" input
+		(pin "~{EN}" input
 			(at 52.07 73.66 180)
 			(effects
@@
 			)
 		)
-		(pin "CK" input
+		(pin "~{EN}" input
 			(at 134.62 38.1 180)
 			(effects
@@
 			)
 		)
-		(pin "CK" input
+		(pin "~{EN}" input
 			(at 52.07 113.03 180)
 			(effects
@@
 			)
 		)
-		(pin "CK" input
-			(at 52.07 58.42 180)
-			(effects
-				(font
-					(size 1.27 1.27)
-				)
-				(justify left)
-			)
-		)
 		(pin "D[0..15]" input
 			(at 52.07 55.88 180)
@@
 				)
 				(justify right)
+			)
+		)
+		(pin "~{EN}" input
+			(at 52.07 58.42 180)
+			(effects
+				(font
+					(size 1.27 1.27)
+				)
+				(justify left)
 			)
 		)
@@
 			)
 		)
-		(pin "CK" input
-			(at 87.63 44.45 180)
-			(effects
-				(font
-					(size 1.27 1.27)
-				)
-				(justify left)
-			)
-		)
 		(pin "~{INC}" input
 			(at 87.63 41.91 180)
@@
 			)
 		)
-		(pin "CK" input
+		(pin "~{EN}" input
 			(at 52.07 90.17 180)
 			(effects
@@
 				)
 			)
+		)
+	)
+	(sheet
+		(at 167.64 33.02)
+		(size 20.32 35.56)
+		(exclude_from_sim no)
+		(in_bom yes)
+		(on_board yes)
+		(dnp no)
+		(stroke
+			(width 0.1524)
+			(type solid)
+		)
+		(fill
+			(color 0 0 0 0)
+		)
+		(property "Sheetname" "uSEQ"
+			(at 171.704 40.132 0)
+			(show_name no)
+			(do_not_autoplace no)
+			(effects
+				(font
+					(size 2.54 2.54)
+				)
+				(justify left bottom)
+			)
+		)
+		(property "Sheetfile" "decode.kicad_sch"
+			(at 167.64 69.596 0)
+			(show_name no)
+			(do_not_autoplace no)
+			(effects
+				(font
+					(size 1.27 1.27)
+				)
+				(justify left top)
+			)
+		)
+		(pin "D[0..15]" input
+			(at 167.64 35.56 180)
+			(effects
+				(font
+					(size 1.27 1.27)
+				)
+				(justify left)
+			)
+		)
+		(instances
+			(project "CPU"
+				(path "/a20f94c8-e12f-422f-aacc-6eccc92eb74d"
+					(page "10")
+				)
+			)
