File: KiCAD/CPU/PC.kicad_sch (KiCad schematic)
At the start: 6 parts, among them U1 74LS163, U2 74LS163, U3 74LS163, U4 74LS163, U5 74LS244, U6 74LS244

Commit message: small updates
Connections:
- net CK renamed CLK
Changed lines of the file:
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@@
+		)
+	)
+	(global_label "CLK"
+		(shape input)
+		(at 38.1 62.23 180)
+		(fields_autoplaced yes)
+		(effects
+			(font
+				(size 1.27 1.27)
+			)
+			(justify right)
+		)
+		(property "Intersheetrefs" "${INTERSHEET_REFS}"
+			(at 31.5467 62.23 0)
+			(hide yes)
+			(show_name no)
+			(do_not_autoplace no)
+			(effects
+				(font
+					(size 1.27 1.27)
+				)
+				(justify right)
+			)
 		)
 	)
@@
 		(effects
 			(font
-				(size 1.27 1.27)
-			)
-			(justify right)
-		)
-	)
-	(hierarchical_label "CK"
-		(shape input)
-		(at 38.1 62.23 180)
-		(effects
-			(font
